File: Anemosens/ANEMOMETRO_PCB/ANEMOMETRO.kicad_pcb (KiCad board)
At the start: 2 copper layers, 8 parts, among them Q1 2N2222A, U3 A3144E

Commit message: Acertando os arquivos
Parts:
- removed Q1 (x2): 2N2222A, Package_TO_SOT_THT:TO-92_Inline_Horizontal2
- removed the R1 at (97.4, 59.1)
- removed the R1 at (114.9, 60.6)
- removed the R2 at (97.4, 69.1)
- removed the R2 at (114.9, 70.8)
- removed U3 (x2): A3144E, Package_TO_SOT_THT:TO-92S
- added C4: 47nF, Capacitor_SMD:C_0805_2012Metric_Pad1.18x1.45mm_HandSolder, F.Cu at (157.2, 145.2)
- added C4: 47nF, Capacitor_SMD:C_0805_2012Metric_Pad1.18x1.45mm_HandSolder, F.Cu at (221.0, 205.8)
- added C4: 47nF, Capacitor_SMD:C_0805_2012Metric_Pad1.18x1.45mm_HandSolder, F.Cu at (221.2, 144.8)
- added C4: 47nF, Capacitor_SMD:C_0805_2012Metric_Pad1.18x1.45mm_HandSolder, F.Cu at (274.8, 203.0)
- added C4: 47nF, Capacitor_SMD:C_0805_2012Metric_Pad1.18x1.45mm_HandSolder, F.Cu at (271.5, 146.5)
- added C4: 47nF, Capacitor_SMD:C_0805_2012Metric_Pad1.18x1.45mm_HandSolder, F.Cu at (160.5, 202.0)
- added Q2: MMBT3904, Package_TO_SOT_SMD:SOT-23, F.Cu at (272.8, 154.4)
- added Q2: MMBT3904, Package_TO_SOT_SMD:SOT-23, F.Cu at (158.5, 153.2)
- added Q2: MMBT3904, Package_TO_SOT_SMD:SOT-23, F.Cu at (222.5, 152.7)
- added Q2: MMBT3904, Package_TO_SOT_SMD:SOT-23, F.Cu at (222.2, 213.7)
- added Q2: MMBT3904, Package_TO_SOT_SMD:SOT-23, F.Cu at (161.8, 209.9)
- added Q2: MMBT3904, Package_TO_SOT_SMD:SOT-23, F.Cu at (276.0, 210.9)
- added R1: 0R_0603, Resistor_SMD:R_1206_3216Metric_Pad1.30x1.75mm_HandSolder, F.Cu at (221.5, 209.5)
- added R1: 0R_0603, Resistor_SMD:R_1206_3216Metric_Pad1.30x1.75mm_HandSolder, F.Cu at (157.8, 149.0)
- added R1: 0R_0603, Resistor_SMD:R_1206_3216Metric_Pad1.30x1.75mm_HandSolder, F.Cu at (221.8, 148.5)
- added R1: 0R_0603, Resistor_SMD:R_1206_3216Metric_Pad1.30x1.75mm_HandSolder, F.Cu at (275.2, 206.8)
- added R1: 0R_0603, Resistor_SMD:R_1206_3216Metric_Pad1.30x1.75mm_HandSolder, F.Cu at (161.0, 205.8)
- added R1: 0R_0603, Resistor_SMD:R_1206_3216Metric_Pad1.30x1.75mm_HandSolder, F.Cu at (272.0, 150.2)
- added R2: 0R_0603, Resistor_SMD:R_1206_3216Metric_Pad1.30x1.75mm_HandSolder, F.Cu at (275.2, 216.8)
- added R2: 0R_0603, Resistor_SMD:R_1206_3216Metric_Pad1.30x1.75mm_HandSolder, F.Cu at (221.8, 158.5)
- added R2: 0R_0603, Resistor_SMD:R_1206_3216Metric_Pad1.30x1.75mm_HandSolder, F.Cu at (161.0, 215.8)
- added R2: 0R_0603, Resistor_SMD:R_1206_3216Metric_Pad1.30x1.75mm_HandSolder, F.Cu at (272.0, 160.2)
- added R2: 0R_0603, Resistor_SMD:R_1206_3216Metric_Pad1.30x1.75mm_HandSolder, F.Cu at (157.8, 159.0)
- added R2: 0R_0603, Resistor_SMD:R_1206_3216Metric_Pad1.30x1.75mm_HandSolder, F.Cu at (221.5, 219.5)
- added U2: A3144E, Package_TO_SOT_THT:TO-92S, F.Cu at (220.2, 202.7)
- added U2: A3144E, Package_TO_SOT_THT:TO-92S, F.Cu at (159.8, 198.9)
- added U2: A3144E, Package_TO_SOT_THT:TO-92S, F.Cu at (156.5, 142.2)
- added U2: A3144E, Package_TO_SOT_THT:TO-92S, F.Cu at (274.0, 199.9)
- added U2: A3144E, Package_TO_SOT_THT:TO-92S, F.Cu at (220.5, 141.7)
- added U2: A3144E, Package_TO_SOT_THT:TO-92S, F.Cu at (270.8, 143.4)
Routing:
- net Net-(Q2-B): track 0.00 -> 63.9 mm
- net GND: track 39.1 -> 0.00 mm
- net OUT: track 11.2 -> 49.7 mm, vias 0 -> 6
- net Net-(Q1-B): track 28.8 -> 0.00 mm
- net +5V: track 119.4 -> 122.6 mm, vias 0 -> 6
- net Earth: vias 0 -> 6
- added copper zone on F.Cu, net Earth
- removed copper zone on F.Cu, net +5V
- removed copper zone on F.Cu, net GND
Other:
- board outline added: 122.5 x 84 mm
