File: Anemosens/ANEMOMETRO_PCB/ANEMOMETRO.kicad_sch (KiCad schematic)
At the start: 11 parts, among them J1 Conn_01x08_Pin, Q1 2N2222A, U1 AMS1117-5.0, U2 AS5600, U3 A3144E

Commit message: Acertando os arquivos
Parts:
- removed C2: 10uF, Capacitor_SMD:C_0805_2012Metric_Pad1.18x1.45mm_HandSolder, symbol Device:C
- removed Q1: 2N2222A, Package_TO_SOT_THT:TO-92_Inline_Horizontal2, symbol PCM_Transistor_BJT_AKL:2N2222A
- removed U2: AS5600, PCM_4ms_Package_SOIC:SOIC-8_3.9x4.9mm_Pitch1.27mm, symbol Sensor_Magnetic:AS5045B
- added C4: 47nF, Capacitor_SMD:C_0805_2012Metric_Pad1.18x1.45mm_HandSolder, symbol PCM_Elektuur:C
- added Q2: MMBT3904, Package_TO_SOT_SMD:SOT-23, symbol PCM_Transistor_BJT_AKL:MMBT3904
- R1, R2: footprint PCM_Resistor_THT_US_AKL_Double:R_Axial_DIN0204_L3.6mm_D1.6mm_P7.62mm_Horizontal -> Resistor_SMD:R_1206_3216Metric_Pad1.30x1.75mm_HandSolder
- renumbered C3 to C2, C4 to C3, U3 to U2
Connections:
- net Earth: now also C4.2 (-), Q2.2 (E); no longer R1.1, R2.1, U2.1 (VCC)
- net OUT: now also Q2.3 (C)
- net at R1.2, U2.3 (OUT): now also Q2.1 (B)
- new net +5V: C4.1 (+), R1.1, R2.1, U2.1 (VCC)
Other:
- moved on the sheet: J1
